File: HW/electronics/electronics.kicad_sch (KiCad schematic)
At the start: 41 parts, among them J1 RADIO, J10 CR2032 socket, J11 AAA socket, J12 AA Socket, J13 RAW IN, J2 DCDC converter, J3 I2C Sensor (BME/BMP 280), J4 PWM out, J5 OneWire sensor, J6 ISP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

Commit message: placa completa
Parts:
- removed C1, C4: 10u, Capacitor_THT:CP_Radial_D5.0mm_P2.50mm, symbol Device:CP
- removed C2: 100n, Capacitor_THT:C_Rect_L7.0mm_W2.0mm_P5.00mm, symbol Device:C
- removed C3: 1u, Capacitor_THT:CP_Radial_D4.0mm_P1.50mm, symbol Device:CP1
- removed C5: 1n, Capacitor_THT:CP_Radial_Tantal_D4.5mm_P2.50mm, symbol Device:C
- removed C6: 0.1u, Capacitor_THT:CP_Radial_Tantal_D4.5mm_P2.50mm, symbol Device:CP
- removed D1: LED, LED_THT:LED_D1.8mm_W3.3mm_H2.4mm, symbol Device:LED
- removed D2, D3: 1N914, Diode_THT:D_DO-35_SOD27_P7.62mm_Horizontal, symbol Diode:1N914
- removed J1: RADIO, Connector_PinHeader_2.54mm:PinHeader_1x03_P2.54mm_Vertical, symbol Connector:Conn_01x03_Male
- removed J10: CR2032 socket, battery supp.:BatteryHolder_Keystone_106_1x21mm, symbol Connector:Screw_Terminal_01x02
- removed J11: AAA socket, Battery:BatteryHolder_Keystone_2466_1xAAA, symbol Connector:Screw_Terminal_01x02
- removed J12: AA Socket, Battery:BatteryHolder_Keystone_2460_1xAA, symbol Connector:Screw_Terminal_01x02
- removed J13: RAW IN, TerminalBlock:TerminalBlock_bornier-2_P5.08mm, symbol Connector:Screw_Terminal_01x02
- removed J2: DCDC converter, TinySensor lib:DC-DC_0.9v-3.3v_to_3.3v, symbol Connector_Generic:Conn_01x03
- removed J4: PWM out, Connector_PinHeader_2.54mm:PinHeader_1x02_P2.54mm_Vertical, symbol Connector:Conn_01x02_Male
- removed J5: OneWire sensor, Connector_PinHeader_2.54mm:PinHeader_1x03_P2.54mm_Vertical, symbol Connector_Generic:Conn_01x03
- removed J6: ISP, TinySensor lib:ICSP_SOCKET_MINI_2x3, symbol tinySensorv1-rescue:AVR-ISP-6-Connector
- removed J7: Analog sensor, Connector_PinHeader_2.54mm:PinHeader_1x03_P2.54mm_Vertical, symbol Connector_Generic:Conn_01x03
- removed J8: EXT. INT0, Connector_PinHeader_2.54mm:PinHeader_1x02_P2.54mm_Vertical, symbol Connector_Generic:Conn_01x02
- removed JP1: LED Jumper, Connector_PinHeader_2.54mm:PinHeader_1x02_P2.54mm_Vertical, symbol Device:Jumper
- removed JP2: DIRECT Vcc, Jumper:SolderJumper-2_P1.3mm_Open_TrianglePad1.0x1.5mm, symbol Jumper:SolderJumper_2_Open
- removed JP3: (no value), Jumper:SolderJumper-2_P1.3mm_Open_TrianglePad1.0x1.5mm, symbol Jumper:SolderJumper_2_Open
- removed JP4: Analog ref, Jumper:SolderJumper-3_P1.3mm_Open_Pad1.0x1.5mm_NumberLabels, symbol Jumper:SolderJumper_3_Open
- removed MH1, MH2, MH3, MH4, MH5, MH6: MountingHole, MountingHole:MountingHole_2.5mm, symbol Mechanical:MountingHole
- removed R1: 1k, Resistor_THT:R_Axial_DIN0204_L3.6mm_D1.6mm_P7.62mm_Horizontal, symbol Device:R
- removed R2, R3: 4,7k, Resistor_THT:R_Axial_DIN0204_L3.6mm_D1.6mm_P7.62mm_Horizontal, symbol Device:R
- removed R4: 75R, Resistor_THT:R_Axial_DIN0204_L3.6mm_D1.6mm_P7.62mm_Horizontal, symbol Device:R
- removed R5: 10k, Resistor_THT:R_Axial_DIN0204_L3.6mm_D1.6mm_P7.62mm_Horizontal, symbol Device:R
- removed R6, R7: 4k7, Resistor_THT:R_Axial_DIN0204_L3.6mm_D1.6mm_P7.62mm_Horizontal, symbol Device:R
- removed SW1: RESET, Button_Switch_THT:SW_PUSH_6mm_H4.3mm, symbol Switch:SW_Push
- removed U1: ATtiny84A-PU, Package_DIP:DIP-14_W7.62mm, symbol tinySensorv1-rescue:ATtiny84A-PU-MCU_Microchip_ATtiny-tinySensorv1-rescue
- added J2: 4ch relay, TinySensor lib:BMx280_breakout, symbol Connector:Conn_01x06_Female
- added PS?: HLK-PM01, Converter_ACDC:Converter_ACDC_HiLink_HLK-PMxx, symbol Converter_ACDC:HLK-PM01
- added U2: ESP32-MB, ESP32-CAM, symbol ESP32-CAM:ESP32-CAM
- gave numbers to parts that had none: 1
Connections:
- net SENSOR_VCC is gone; now on net SDA: J3.1 (Pin_1)
- net GND: now also U1.16 (GND_3), U1.7 (GND_1), J2.1 (Pin_1), PS?.3 (-Vout), U2.16 (GND_3); no longer J3.2 (Pin_2), J3.6 (Pin_6)
- net SCL: now also J3.2 (Pin_2), U1.11 (IO0); no longer J3.3 (Pin_3)
- net SDA: now also U1.10 (IO16); no longer J3.4 (Pin_4)
- net at U1.12 (GND_2): now also J3.3 (Pin_3)
- net at U1.13 (VCC): now also J3.4 (Pin_4)
- net at U1.14 (U0R): now also U2.14 (U0R)
- net at U1.15 (U0T): now also U2.15 (U0T)
- net at U1.3 (IO14): now also J2.2 (Pin_2)
- net at U1.4 (IO15): now also J2.3 (Pin_3)
- net +5V: now reaches U1.8 (5V)
- net +5V: now also J2.6 (Pin_6), PS?.4 (+Vout)
Other:
- note removed: "(and MOSI)"
- note removed: "(and SCK)"
- note removed: "433Mhz emitter connection"
- note removed: "Bypass of DC-DC converter"
- note removed: "CSB"
- note removed: "I2C bus pullups"
- note removed: "LM35 below 0° circuitry"
- note removed: "Optional"
- note removed: "Optional RC filter for LM35 sensor or resistor bridge for LDR"
- note removed: "Power management"
- note removed: "R4 == 18k if used with LM35 "below 0°" setup"
- note removed: "Radio activity led"
- note removed: "SDO"
- note removed: "Sensors connections"
- company: (none) -> Altermundi // INTI
- title: TinySensor board -> Libre Pollo
- moved on the sheet: U1

Commit message: addedvaristor
Parts:
- added J1: 220 v in, symbol Connector:Screw_Terminal_01x02
- added RV?: Varistor, symbol Device:Varistor
Connections:
- net at PS?.1 (AC/L): now also J1.2 (Pin_2), RV?.1
- net at PS?.2 (AC/N): now also J1.1 (Pin_1), RV?.2
Changed lines of the file:
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@@
   (junction (at 203.2 76.2) (diameter 0) (color 0 0 0 0)
+  )
+  (junction (at 138.43 92.71) (diameter 0) (color 0 0 0 0)
+  )
+  (junction (at 138.43 85.09) (diameter 0) (color 0 0 0 0)
   )
   (junction (at 245.11 134.62) (diameter 0) (color 0 0 0 0)
@@
     (stroke (width 0) (type default) (color 0 0 0 0))
   )
+  (wire (pts (xy 149.86 90.17) (xy 149.86 92.71))
+    (stroke (width 0) (type default) (color 0 0 0 0))
+  )
   (wire (pts (xy 241.3 130.81) (xy 241.3 127))
     (stroke (width 0) (type default) (color 0 0 0 0))
@@
     (stroke (width 0) (type default) (color 0 0 0 0))
   )
+  (wire (pts (xy 138.43 85.09) (xy 153.67 85.09))
+    (stroke (width 0) (type default) (color 0 0 0 0))
+  )
   (wire (pts (xy 240.03 125.73) (xy 240.03 118.11))
     (stroke (width 0) (type default) (color 0 0 0 0))
@@
     (stroke (width 0) (type default) (color 0 0 0 0))
   )
+  (wire (pts (xy 125.73 87.63) (xy 133.35 87.63))
+    (stroke (width 0) (type default) (color 0 0 0 0))
+  )
   (wire (pts (xy 200.66 113.03) (xy 205.74 113.03))
     (stroke (width 0) (type default) (color 0 0 0 0))
@@
     (stroke (width 0) (type default) (color 0 0 0 0))
   )
+  (wire (pts (xy 149.86 92.71) (xy 138.43 92.71))
+    (stroke (width 0) (type default) (color 0 0 0 0))
+  )
   (wire (pts (xy 173.99 90.17) (xy 176.53 90.17))
     (stroke (width 0) (type default) (color 0 0 0 0))
   )
+  (wire (pts (xy 125.73 85.09) (xy 138.43 85.09))
+    (stroke (width 0) (type default) (color 0 0 0 0))
+  )
   (wire (pts (xy 184.15 125.73) (xy 205.74 125.73))
     (stroke (width 0) (type default) (color 0 0 0 0))
@@
     (stroke (width 0) (type default) (color 0 0 0 0))
   )
+  (wire (pts (xy 133.35 87.63) (xy 133.35 92.71))
+    (stroke (width 0) (type default) (color 0 0 0 0))
+  )
   (wire (pts (xy 203.2 76.2) (xy 203.2 110.49))
     (stroke (width 0) (type default) (color 0 0 0 0))
@@
     (stroke (width 0) (type default) (color 0 0 0 0))
   )
+  (wire (pts (xy 153.67 90.17) (xy 149.86 90.17))
+    (stroke (width 0) (type default) (color 0 0 0 0))
+  )
   (wire (pts (xy 195.58 81.28) (xy 195.58 115.57))
     (stroke (width 0) (type default) (color 0 0 0 0))
   )
   (wire (pts (xy 184.15 118.11) (xy 205.74 118.11))
+    (stroke (width 0) (type default) (color 0 0 0 0))
+  )
+  (wire (pts (xy 133.35 92.71) (xy 138.43 92.71))
     (stroke (width 0) (type default) (color 0 0 0 0))
   )
@@
     (pin "3")
     (pin "4")
+  )
+  (symbol (lib_id "Connector:Screw_Terminal_01x02") (at 120.65 87.63 180) (unit 1)
+    (in_bom yes) (on_board yes) (fields_autoplaced)
+    (property "Reference" "J1" (id 0) (at 120.65 78.74 0))
+    (property "Value" "220 v in" (id 1) (at 120.65 81.28 0))
+    (property "Footprint" "" (id 2) (at 120.65 87.63 0)
+      (effects (font (size 1.27 1.27)) hide)
+    )
+    (property "Datasheet" "~" (id 3) (at 120.65 87.63 0)
+      (effects (font (size 1.27 1.27)) hide)
+    )
+    (pin "1")
+    (pin "2")
   )
   (symbol (lib_id "ESP32-CAM:ESP32-CAM") (at 237.49 93.98 180) (unit 1)
@@
     (pin "9")
   )
+  (symbol (lib_id "Device:Varistor") (at 138.43 88.9 0) (unit 1)
+    (in_bom yes) (on_board yes) (fields_autoplaced)
+    (property "Reference" "RV?" (id 0) (at 140.97 87.8831 0)
+      (effects (font (size 1.27 1.27)) (justify left))
+    )
+    (property "Value" "Varistor" (id 1) (at 140.97 90.4231 0)
+      (effects (font (size 1.27 1.27)) (justify left))
+    )
+    (property "Footprint" "" (id 2) (at 136.652 88.9 90)
+      (effects (font (size 1.27 1.27)) hide)
+    )
+    (property "Datasheet" "~" (id 3) (at 138.43 88.9 0)
+      (effects (font (size 1.27 1.27)) hide)
+    )
+    (pin "1")
+    (pin "2")
+  )
   (symbol (lib_id "power:GND") (at 246.38 111.76 180) (unit 1)
     (in_bom yes) (on_board yes) (fields_autoplaced)
@@
       (reference "#PWR?") (unit 1) (value "GND") (footprint "")
     )
+    (path "/3b5c237f-d7d6-49ed-b03e-6a11bbbe8b45"
+      (reference "J1") (unit 1) (value "220 v in") (footprint "")
+    )
     (path "/e260159f-6319-49b0-9353-32ce1409520f"
       (reference "J2") (unit 1) (value "4ch relay") (footprint "TinySensor lib:BMx280_breakout")
@@
       (reference "PS?") (unit 1) (value "HLK-PM01") (footprint "Converter_ACDC:Converter_ACDC_HiLink_HLK-PMxx")
     )
+    (path "/5bb32dcb-8a97-4374-8a16-bc17822d4db3"
+      (reference "RV?") (unit 1) (value "Varistor") (footprint "")
+    )
     (path "/e092ad44-1d6c-49d8-a179-c78eb33d229b"
